Commit message: baguete

File: src/assets/skateboard/robot.urdf (robot description, URDF)
Before this commit: robot robot, 7 links, 6 joints
Links:
- link base_link: geometry collision mesh filename=meshes/base_link.STL; visual mesh filename=meshes/base_link.STL
- link tr0: geometry collision mesh filename=meshes/tr0.STL; visual mesh filename=meshes/tr0.STL
- link tr1: geometry collision mesh filename=meshes/tr1.STL; visual mesh filename=meshes/tr1.STL
- link wh0: geometry collision mesh filename=meshes/wh0.STL; visual mesh filename=meshes/wh0.STL
- link wh1: geometry collision mesh filename=meshes/wh1.STL; visual mesh filename=meshes/wh1.STL
- link wh2: geometry collision mesh filename=meshes/wh2.STL; visual mesh filename=meshes/wh2.STL
- link wh3: geometry collision mesh filename=meshes/wh3.STL; visual mesh filename=meshes/wh3.STL
